File: OpenC64KernalCart.sch (KiCad schematic (older format))
At the start: 11 parts, among them J1 C64-Exp-Port, J2 CPU_WIRE, J3 CONN_3X2, J97 TOP_TRACKS, J98 BOTTOM_TRACKS, J99 OSHW_LOGO, SW1 KERNEL_BANK, U1 27128, U2 74LS30

Commit message: Sukko's Version 1
Parts:
- removed J3: CONN_3X2, Connector_PinHeader_2.54mm:PinHeader_2x03_P2.54mm_Vertical, symbol conn:CONN_3X2
- removed R1: R, Resistor_THT:R_Axial_DIN0207_L6.3mm_D2.5mm_P10.16mm_Horizontal, symbol Device:R
- added SW2: RESET_SWITCH, OpenC64KernalCart:PCB_PUSH, symbol Switch:SW_DIP_x02
- J2: footprint Connector_PinHeader_2.54mm:PinHeader_1x01_P2.54mm_Vertical -> OpenC64KernalCart:PinHeader_1x01_P2.54mm_Vertical
- U1: footprint Package_DIP:DIP-28_W15.24mm -> Package_DIP:DIP-28_W15.24mm_Socket_LongPads
Connections:
- wire segments 116 -> 112
Changed lines of the file:
@@
 Text Label 6420 5830 0    50   ~ 0
 a13x
-$Comp
-L Device:R R1
-U 1 1 5CEF88EE
-P 7365 5555
-F 0 "R1" H 7435 5601 50  0000 L CNN
-F 1 "R" H 7435 5510 50  0000 L CNN
-F 2 "Resistor_THT:R_Axial_DIN0207_L6.3mm_D2.5mm_P10.16mm_Horizontal" V 7295 5555 50  0001 C CNN
-F 3 "~" H 7365 5555 50  0001 C CNN
-	1    7365 5555
-	1    0    0    -1
-$EndComp
-$Comp
-L power:VCC #PWR0107
-U 1 1 5CEF8EB6
-P 7365 5265
-F 0 "#PWR0107" H 7365 5115 50  0001 C CNN
-F 1 "VCC" H 7382 5438 50  0000 C CNN
-F 2 "" H 7365 5265 50  0001 C CNN
-F 3 "" H 7365 5265 50  0001 C CNN
-	1    7365 5265
-	1    0    0    -1
-$EndComp
-Wire Wire Line
-	7365 5265 7365 5405
-Wire Wire Line
-	7365 5780 7365 5705
 Wire Wire Line
 	6950 5780 7365 5780
@@
 F 0 "J2" H 4868 5659 50  0000 R CNN
 F 1 "CPU_WIRE" H 4868 5568 50  0000 R CNN
-F 2 "Connector_PinHeader_2.54mm:PinHeader_1x01_P2.54mm_Vertical" H 4895 5635 50  0001 C CNN
+F 2 "OpenC64KernalCart:PinHeader_1x01_P2.54mm_Vertical" H 4895 5635 50  0001 C CNN
 F 3 "~" H 4895 5635 50  0001 C CNN
 	1    4895 5635
@@
 F 0 "U1" H 6875 3685 50  0000 C CNN
 F 1 "27128" H 6925 1585 50  0000 C CNN
-F 2 "Package_DIP:DIP-28_W15.24mm" H 7110 2635 50  0001 C CNN
+F 2 "Package_DIP:DIP-28_W15.24mm_Socket_LongPads" H 7110 2635 50  0001 C CNN
 F 3 "http://eeshop.unl.edu/pdf/27128.pdf" H 7110 2635 50  0001 C CNN
 	1    7110 2635
@@
 Wire Wire Line
 	10815 785  10815 875
-$Comp
-L conn:CONN_3X2 J3
-U 1 1 5CFA2A39
-P 9900 2710
-F 0 "J3" H 9900 3060 50  0000 C CNN
-F 1 "CONN_3X2" H 9900 2976 40  0000 C CNN
-F 2 "Connector_PinHeader_2.54mm:PinHeader_2x03_P2.54mm_Vertical" H 9900 2710 50  0001 C CNN
-F 3 "" H 9900 2710 50  0001 C CNN
-	1    9900 2710
-	1    0    0    -1
-$EndComp
-Wire Wire Line
-	9500 2560 9405 2560
-Wire Wire Line
-	9500 2760 9405 2760
-Text Label 9040 2560 0    50   ~ 0
-exrom
-Text Label 9040 2660 0    50   ~ 0
+Text Label 9075 2625 0    50   ~ 0
 reset
 Wire Wire Line
-	9405 2560 9405 2760
-Connection ~ 9405 2560
-Wire Wire Line
-	9405 2560 9010 2560
-Wire Wire Line
-	9010 2660 9500 2660
+	9045 2625 9360 2625
 $Comp
 L power:GND #PWR0112
 U 1 1 5CFBF7DF
-P 10455 2900
-F 0 "#PWR0112" H 10455 2650 50  0001 C CNN
-F 1 "GND" H 10460 2727 50  0000 C CNN
-F 2 "" H 10455 2900 50  0001 C CNN
-F 3 "" H 10455 2900 50  0001 C CNN
-	1    10455 2900
-	-1   0    0    -1
-$EndComp
-Wire Wire Line
-	10455 2760 10455 2900
-Connection ~ 10455 2760
-Wire Wire Line
-	10455 2760 10300 2760
-Wire Wire Line
-	10455 2760 10455 2660
-Wire Wire Line
-	10455 2560 10300 2560
-Connection ~ 10455 2660
-Wire Wire Line
-	10455 2660 10300 2660
-Wire Wire Line
-	10455 2660 10455 2560
+P 10290 2765
+F 0 "#PWR0112" H 10290 2515 50  0001 C CNN
+F 1 "GND" H 10295 2592 50  0000 C CNN
+F 2 "" H 10290 2765 50  0001 C CNN
+F 3 "" H 10290 2765 50  0001 C CNN
+	1    10290 2765
+	-1   0    0    -1
+$EndComp
+Wire Wire Line
+	10290 2625 10290 2765
+Connection ~ 10290 2625
+Wire Wire Line
+	10290 2625 10135 2625
+Wire Wire Line
+	10290 2625 10290 2525
 NoConn ~ 1800 2515
 $Comp
@@
 Wire Wire Line
 	9270 5865 9270 6000
+$Comp
+L Switch:SW_DIP_x02 SW2
+U 1 1 5CE467F2
+P 9835 2625
+F 0 "SW2" H 9835 2992 50  0000 C CNN
+F 1 "RESET_SWITCH" H 9835 2901 50  0000 C CNN
+F 2 "OpenC64KernalCart:PCB_PUSH" H 9835 2625 50  0001 C CNN
+F 3 "~" H 9835 2625 50  0001 C CNN
+	1    9835 2625
+	1    0    0    -1
+$EndComp
+Wire Wire Line
+	10135 2525 10290 2525
+Wire Wire Line
+	9535 2525 9360 2525
+Wire Wire Line
+	9360 2525 9360 2625
+Connection ~ 9360 2625
+Wire Wire Line
+	9360 2625 9535 2625
+Wire Wire Line
+	7365 5780 7365 5625
+$Comp
+L power:VCC #PWR0107
+U 1 1 5CEF8EB6
+P 7365 5625
+F 0 "#PWR0107" H 7365 5475 50  0001 C CNN
+F 1 "VCC" H 7382 5798 50  0000 C CNN
+F 2 "" H 7365 5625 50  0001 C CNN
+F 3 "" H 7365 5625 50  0001 C CNN
+	1    7365 5625
+	1    0    0    -1
+$EndComp
 Wire Bus Line
 	1380 2715 1380 3415

Commit message: Ready for Sukko's V1
Parts:
- removed U1: 27128, Package_DIP:DIP-28_W15.24mm_Socket_LongPads, symbol Memory_EPROM:27128
- added C2: 100n, Capacitor_THT:C_Disc_D7.5mm_W2.5mm_P5.00mm, symbol Device:C
- added SW13: KERNEL_BANK_A13, OpenC64KernalCart:Switch, symbol w_device:SW_SPDT
- added SW14: KERNEL_BANK_A14, OpenC64KernalCart:Switch, symbol w_device:SW_SPDT
- added U1: 27512, Package_DIP:DIP-28_W15.24mm_Socket_LongPads, symbol Memory_EPROM:27512
- SW15: renamed from SW1; value KERNEL_BANK -> KERNEL_BANK_A15
Connections:
- net labels added: a14x, a15x
- wire segments 112 -> 129
- no-connect marks 10 -> 11
Other:
- moved on the sheet: C1, SW15
Changed lines of the file:
@@
 Sheet 1 1
 Title "OpenC64KernalCart"
-Date "2019-05-20"
-Rev "1git"
+Date "2019-05-22"
+Rev "1"
 Comp "SukkoPera"
 Comment1 "Licensed under CERN OHL v.1.2"
@@
 game
 $Comp
-L w_device:SW_SPDT SW1
+L w_device:SW_SPDT SW15
 U 1 1 5CEE37BE
-P 6800 5830
-F 0 "SW1" H 6800 6061 50  0000 C CNN
-F 1 "KERNEL_BANK" H 6800 5695 50  0000 C CNN
-F 2 "OpenC64KernalCart:Switch" H 6800 5830 60  0001 C CNN
-F 3 "" H 6800 5830 60  0000 C CNN
-	1    6800 5830
-	1    0    0    -1
-$EndComp
-Wire Wire Line
-	6650 5830 6385 5830
-Text Label 6420 5830 0    50   ~ 0
-a13x
-Wire Wire Line
-	6950 5780 7365 5780
+P 8300 5875
+F 0 "SW15" H 8300 6106 50  0000 C CNN
+F 1 "KERNEL_BANK_A15" H 8300 5740 50  0000 C CNN
+F 2 "OpenC64KernalCart:Switch" H 8300 5875 60  0001 C CNN
+F 3 "" H 8300 5875 60  0000 C CNN
+	1    8300 5875
+	1    0    0    -1
+$EndComp
+Wire Wire Line
+	8150 5875 7885 5875
+Text Label 7920 5875 0    50   ~ 0
+a15x
+Wire Wire Line
+	8450 5825 8865 5825
 $Comp
 L power:GND #PWR0108
 U 1 1 5CF018BC
-P 7365 6015
-F 0 "#PWR0108" H 7365 5765 50  0001 C CNN
-F 1 "GND" H 7370 5842 50  0000 C CNN
-F 2 "" H 7365 6015 50  0001 C CNN
-F 3 "" H 7365 6015 50  0001 C CNN
-	1    7365 6015
+P 8865 6060
+F 0 "#PWR0108" H 8865 5810 50  0001 C CNN
+F 1 "GND" H 8870 5887 50  0000 C CNN
+F 2 "" H 8865 6060 50  0001 C CNN
+F 3 "" H 8865 6060 50  0001 C CNN
+	1    8865 6060
 	-1   0    0    -1
 $EndComp
 Wire Wire Line
-	6950 5880 7365 5880
-Wire Wire Line
-	7365 5880 7365 6015
+	8450 5925 8865 5925
+Wire Wire Line
+	8865 5925 8865 6060
 Text Label 5130 5635 0    50   ~ 0
 wire
@@
 	0    1    1    0
 $EndComp
-$Comp
-L Memory_EPROM:27128 U1
-U 1 1 5CF35B9C
-P 7110 2635
-F 0 "U1" H 6875 3685 50  0000 C CNN
-F 1 "27128" H 6925 1585 50  0000 C CNN
-F 2 "Package_DIP:DIP-28_W15.24mm_Socket_LongPads" H 7110 2635 50  0001 C CNN
-F 3 "http://eeshop.unl.edu/pdf/27128.pdf" H 7110 2635 50  0001 C CNN
-	1    7110 2635
-	-1   0    0    -1
-$EndComp
-Wire Wire Line
-	7510 3235 7765 3235
-Text Label 7570 3235 0    50   ~ 0
-rw
 Wire Wire Line
 	7510 3435 7765 3435
@@
 Text Label 7570 3535 0    50   ~ 0
 game
-Wire Wire Line
-	7865 3335 7865 3215
-$Comp
-L power:VCC #PWR0109
-U 1 1 5CF5D5F2
-P 7865 3215
-F 0 "#PWR0109" H 7865 3065 50  0001 C CNN
-F 1 "VCC" H 7882 3388 50  0000 C CNN
-F 2 "" H 7865 3215 50  0001 C CNN
-F 3 "" H 7865 3215 50  0001 C CNN
-	1    7865 3215
-	-1   0    0    -1
-$EndComp
-Wire Wire Line
-	7510 3335 7865 3335
 NoConn ~ 10470 6070
 $Comp
@@
 L power:VCC #PWR0114
 U 1 1 5CE3BF1F
-P 9270 5425
-F 0 "#PWR0114" H 9270 5275 50  0001 C CNN
-F 1 "VCC" H 9287 5598 50  0000 C CNN
-F 2 "" H 9270 5425 50  0001 C CNN
-F 3 "" H 9270 5425 50  0001 C CNN
-	1    9270 5425
-	1    0    0    -1
-$EndComp
-Wire Wire Line
-	9270 5425 9270 5565
+P 10670 4380
+F 0 "#PWR0114" H 10670 4230 50  0001 C CNN
+F 1 "VCC" H 10687 4553 50  0000 C CNN
+F 2 "" H 10670 4380 50  0001 C CNN
+F 3 "" H 10670 4380 50  0001 C CNN
+	1    10670 4380
+	1    0    0    -1
+$EndComp
+Wire Wire Line
+	10670 4380 10670 4440
 $Comp
 L Device:C C1
 U 1 1 5CE41467
-P 9270 5715
-F 0 "C1" H 9385 5761 50  0000 L CNN
-F 1 "100n" H 9385 5670 50  0000 L CNN
-F 2 "Capacitor_THT:C_Disc_D7.5mm_W2.5mm_P5.00mm" H 9308 5565 50  0001 C CNN
-F 3 "~" H 9270 5715 50  0001 C CNN
-	1    9270 5715
+P 10460 4670
+F 0 "C1" H 10575 4716 50  0000 L CNN
+F 1 "100n" H 10575 4625 50  0000 L CNN
+F 2 "Capacitor_THT:C_Disc_D7.5mm_W2.5mm_P5.00mm" H 10498 4520 50  0001 C CNN
+F 3 "~" H 10460 4670 50  0001 C CNN
+	1    10460 4670
 	1    0    0    -1
 $EndComp
@@
 L power:GND #PWR0115
 U 1 1 5CE41DD1
-P 9270 6000
-F 0 "#PWR0115" H 9270 5750 50  0001 C CNN
-F 1 "GND" H 9275 5827 50  0000 C CNN
-F 2 "" H 9270 6000 50  0001 C CNN
-F 3 "" H 9270 6000 50  0001 C CNN
-	1    9270 6000
+P 10670 4955
+F 0 "#PWR0115" H 10670 4705 50  0001 C CNN
+F 1 "GND" H 10675 4782 50  0000 C CNN
+F 2 "" H 10670 4955 50  0001 C CNN
+F 3 "" H 10670 4955 50  0001 C CNN
+	1    10670 4955
 	-1   0    0    -1
 $EndComp
-Wire Wire Line
-	9270 5865 9270 6000
 $Comp
 L Switch:SW_DIP_x02 SW2
@@
 	9360 2625 9535 2625
 Wire Wire Line
-	7365 5780 7365 5625
+	8865 5825 8865 5670
 $Comp
 L power:VCC #PWR0107
 U 1 1 5CEF8EB6
-P 7365 5625
-F 0 "#PWR0107" H 7365 5475 50  0001 C CNN
-F 1 "VCC" H 7382 5798 50  0000 C CNN
-F 2 "" H 7365 5625 50  0001 C CNN
-F 3 "" H 7365 5625 50  0001 C CNN
-	1    7365 5625
-	1    0    0    -1
-$EndComp
+P 8865 5670
+F 0 "#PWR0107" H 8865 5520 50  0001 C CNN
+F 1 "VCC" H 8882 5843 50  0000 C CNN
+F 2 "" H 8865 5670 50  0001 C CNN
+F 3 "" H 8865 5670 50  0001 C CNN
+	1    8865 5670
+	1    0    0    -1
+$EndComp
+$Comp
+L Memory_EPROM:27512 U1
+U 1 1 5CEF5BE3
+P 7110 2635
+F 0 "U1" H 6875 3690 50  0000 C CNN
+F 1 "27512" H 6930 1575 50  0000 C CNN
+F 2 "Package_DIP:DIP-28_W15.24mm_Socket_LongPads" H 7110 2635 50  0001 C CNN
+F 3 "http://pdf.datasheetcatalog.com/datasheets/120/227190_DS.pdf" H 7110 2635 50  0001 C CNN
+	1    7110 2635
+	-1   0    0    -1
+$EndComp
+Wire Wire Line
+	7510 3135 7765 3135
+Text Label 7570 3135 0    50   ~ 0
+a14x
+Wire Wire Line
+	7510 3235 7765 3235
+Text Label 7570 3235 0    50   ~ 0
+a15x
+$Comp
+L w_device:SW_SPDT SW14
+U 1 1 5CF11A27
+P 8300 4865
+F 0 "SW14" H 8300 5096 50  0000 C CNN
+F 1 "KERNEL_BANK_A14" H 8300 4730 50  0000 C CNN
+F 2 "OpenC64KernalCart:Switch" H 8300 4865 60  0001 C CNN
+F 3 "" H 8300 4865 60  0000 C CNN
+	1    8300 4865
+	1    0    0    -1
+$EndComp
+Wire Wire Line
+	8150 4865 7885 4865
+Text Label 7920 4865 0    50   ~ 0
+a14x
+Wire Wire Line
+	8450 4815 8865 4815
+$Comp
+L power:GND #PWR0109
+U 1 1 5CF11A34
+P 8865 5050
+F 0 "#PWR0109" H 8865 4800 50  0001 C CNN
+F 1 "GND" H 8870 4877 50  0000 C CNN
+F 2 "" H 8865 5050 50  0001 C CNN
+F 3 "" H 8865 5050 50  0001 C CNN
+	1    8865 5050
+	-1   0    0    -1
+$EndComp
+Wire Wire Line
+	8450 4915 8865 4915
+Wire Wire Line
+	8865 4915 8865 5050
+Wire Wire Line
+	8865 4815 8865 4660
+$Comp
+L power:VCC #PWR0116
+U 1 1 5CF11A41
+P 8865 4660
+F 0 "#PWR0116" H 8865 4510 50  0001 C CNN
+F 1 "VCC" H 8882 4833 50  0000 C CNN
+F 2 "" H 8865 4660 50  0001 C CNN
+F 3 "" H 8865 4660 50  0001 C CNN
+	1    8865 4660
+	1    0    0    -1
+$EndComp
+$Comp
+L w_device:SW_SPDT SW13
+U 1 1 5CF258BE
+P 6845 5295
+F 0 "SW13" H 6845 5526 50  0000 C CNN
+F 1 "KERNEL_BANK_A13" H 6845 5160 50  0000 C CNN
+F 2 "OpenC64KernalCart:Switch" H 6845 5295 60  0001 C CNN
+F 3 "" H 6845 5295 60  0000 C CNN
+	1    6845 5295
+	1    0    0    -1
+$EndComp
+Wire Wire Line
+	6695 5295 6430 5295
+Text Label 6465 5295 0    50   ~ 0
+a13x
+Wire Wire Line
+	6995 5245 7410 5245
+$Comp
+L power:GND #PWR0117
+U 1 1 5CF258CB
+P 7410 5480
+F 0 "#PWR0117" H 7410 5230 50  0001 C CNN
+F 1 "GND" H 7415 5307 50  0000 C CNN
+F 2 "" H 7410 5480 50  0001 C CNN
+F 3 "" H 7410 5480 50  0001 C CNN
+	1    7410 5480
+	-1   0    0    -1
+$EndComp
+Wire Wire Line
+	6995 5345 7410 5345
+Wire Wire Line
+	7410 5345 7410 5480
+Wire Wire Line
+	7410 5245 7410 5090
+$Comp
+L power:VCC #PWR0118
+U 1 1 5CF258D8
+P 7410 5090
+F 0 "#PWR0118" H 7410 4940 50  0001 C CNN
+F 1 "VCC" H 7427 5263 50  0000 C CNN
+F 2 "" H 7410 5090 50  0001 C CNN
+F 3 "" H 7410 5090 50  0001 C CNN
+	1    7410 5090
+	1    0    0    -1
+$EndComp
+NoConn ~ 1800 2315
+$Comp
+L Device:C C2
+U 1 1 5CF4C930
+P 10875 4670
+F 0 "C2" H 10990 4716 50  0000 L CNN
+F 1 "100n" H 10990 4625 50  0000 L CNN
+F 2 "Capacitor_THT:C_Disc_D7.5mm_W2.5mm_P5.00mm" H 10913 4520 50  0001 C CNN
+F 3 "~" H 10875 4670 50  0001 C CNN
+	1    10875 4670
+	1    0    0    -1
+$EndComp
+Wire Wire Line
+	10460 4520 10460 4440
+Wire Wire Line
+	10460 4440 10670 4440
+Connection ~ 10670 4440
+Wire Wire Line
+	10670 4440 10875 4440
+Wire Wire Line
+	10875 4440 10875 4520
+Wire Wire Line
+	10460 4895 10670 4895
+Wire Wire Line
+	10460 4820 10460 4895
+Connection ~ 10670 4895
+Wire Wire Line
+	10670 4895 10670 4955
+Wire Wire Line
+	10670 4895 10875 4895
+Wire Wire Line
+	10875 4895 10875 4820
 Wire Bus Line
 	1380 2715 1380 3415
