File: OpenC64KernalCart.kicad_pcb (KiCad board)
At the start: 2 copper layers, 58.4 x 50.8 mm, 11 parts, among them J1 C64-Exp-Port, J2 CPU_WIRE, J3 CONN_3X2, J97 TOP_TRACKS, J98 BOTTOM_TRACKS, J99 OSHW_LOGO, SW1 KERNEL_BANK, U1 27128, U2 74LS30

Commit message: Sukko's Version 1
Parts:
- removed J3: CONN_3X2, Connector_PinHeader_2.54mm:PinHeader_2x03_P2.54mm_Vertical
- removed R1: R, Resistor_THT:R_Axial_DIN0207_L6.3mm_D2.5mm_P10.16mm_Horizontal
- added SW2: RESET_SWITCH, OpenC64KernalCart:PCB_PUSH, F.Cu at (65.5, 84.7)
- J2: footprint Connector_PinHeader_2.54mm:PinHeader_1x01_P2.54mm_Vertical -> OpenC64KernalCart:PinHeader_1x01_P2.54mm_Vertical
- U1: footprint Package_DIP:DIP-28_W15.24mm -> Package_DIP:DIP-28_W15.24mm_Socket_LongPads
- moved C1 41.4 mm to (68.7, 92.0)
- moved J2 9.29 mm to (67.3, 102.2)
- moved J99 2.93 mm to (111.3, 85.3)
Connections:
- J1 pad 9: /exrom -> (no net)
- SW1 pad 2: Net-(R1-Pad2) -> VCC
Routing:
- net GND: track 123.6 -> 32.0 mm, vias 1 -> 79
- net /exrom: track 66.0 -> 0.00 mm
- net /a13: track 36.2 -> 8.00 mm, vias 1 -> 0
- net /romh: track 89.6 -> 69.9 mm, vias 4 -> 0
- net Net-(R1-Pad2): track 17.7 -> 0.00 mm, vias 1 -> 0
- net /wire: track 9.57 -> 20.0 mm
- net (no net): track 8.25 -> 0.00 mm, vias 1 -> 0
- net /a13x: track 49.3 -> 41.0 mm, vias 2 -> 1
- net /rw: track 49.4 -> 43.1 mm, vias 3 -> 0
- net /game: track 45.4 -> 51.5 mm, vias 5 -> 1
- net /ba: track 58.7 -> 64.2 mm
- net /a12: track 30.5 -> 28.6 mm
- net /reset: track 48.0 -> 47.0 mm, vias 4 -> 0
- net VCC: track 100.4 -> 99.8 mm
- added copper zone on B.Cu, net GND
- added copper zone on F.Cu, net GND
Other:
- board text added: "Licensed under CERN OHL v.1.2"
- board text added: "RESET"
- board text added: "V1"
- board text added: "github.com/SukkoPera/OpenC64KernalCart"

Commit message: Ready for Sukko's V1
Parts:
- added C2: 100n, Capacitor_THT:C_Disc_D7.5mm_W2.5mm_P5.00mm, F.Cu at (63.4, 111.3)
- added SW13: KERNEL_BANK_A13, OpenC64KernalCart:Switch, F.Cu at (109.2, 97.1)
- added SW14: KERNEL_BANK_A14, OpenC64KernalCart:Switch, F.Cu at (109.2, 86.9)
- SW15: renamed from SW1; value KERNEL_BANK -> KERNEL_BANK_A15
- U1: value 27128 -> 27512
- moved J99 2.73 mm to (112.5, 82.9)
- moved SW15 1.21 mm to (112.8, 91.9)
Connections:
- SW15 pad 1: /a13x -> /a15x
- U1 pad 1: VCC -> /a15x
- U1 pad 27: /rw -> /a14x
Routing:
- net /a15x: track 0.00 -> 47.5 mm, vias 0 -> 1
- net /a14x: track 0.00 -> 42.1 mm
- net /rw: track 43.1 -> 9.05 mm
- net VCC: track 99.8 -> 118.6 mm
- net /wire: track 20.0 -> 9.91 mm
- net /a13x: track 41.0 -> 46.4 mm
- net GND: track 32.0 -> 35.5 mm, vias 79 -> 81
- net /d1: track 41.7 -> 40.4 mm
- net /romh: track 69.9 -> 70.9 mm
- net /reset: track 47.0 -> 48.1 mm
- net /ba: track 64.2 -> 65.1 mm
- net /d2: track 35.5 -> 34.6 mm
- net /d0: track 48.2 -> 48.8 mm
Other:
- board text added: "A13"
- board text added: "A14"
- board text added: "A15"

Commit message: Some embellishments
Parts:
- moved J99 1.35 mm to (113.4, 83.9)
Routing:
- net GND: track 35.5 -> 32.0 mm, vias 81 -> 73
Other:
- board text added: "TO CPU PIN 28"
Changed lines of the file:
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@@
   (general
     (thickness 1.6)
-    (drawings 19)
-    (tracks 333)
+    (drawings 28)
+    (tracks 321)
     (zones 0)
     (modules 13)
@@
   (title_block
     (title OpenC64KernalCart)
-    (date 2019-05-22)
+    (date 2019-06-26)
     (rev 1)
     (company SukkoPera)
@@
       (rotate (xyz 0 0 0))
     )
+    (model ${P3D_WALTER}/pth_circuits/dil_14-300_socket.wrl
+      (offset (xyz 3.9 -7.6 0))
+      (scale (xyz 1 1 1))
+      (rotate (xyz 0 0 -90))
+    )
   )
   (module OpenC64KernalCart:Switch (layer F.Cu)
@@
   )
   (module Symbol:OSHW-Logo_5.7x6mm_Copper (layer B.Cu)
-    (at 112.522 82.931 180)
+    (at 113.411 83.947 180)
     (descr "Open Source Hardware Logo")
     (tags "Logo OSHW")
@@
     (descr "C, Disc series, Radial, pin pitch=5.00mm, , diameter*width=7.5*2.5mm^2, Capacitor, http://www.vishay.com/docs/28535/vy2series.pdf")
     (tags "C Disc series Radial pin pitch 5.00mm  diameter 7.5mm width 2.5mm Capacitor")
-    (fp_text reference C1 (at 2.500001 2.54 90) (layer F.SilkS)
+    (fp_text reference C1 (at 2.500001 0.0254 90) (layer F.SilkS)
       (effects (font (size 1 1) (thickness 0.15)))
     )
@@
     (pad 3 thru_hole circle (at 2.25044 3.2512 90) (size 1.99898 1.99898) (drill 1.00076) (layers *.Cu *.Mask F.SilkS)
       (net 1 GND))
-    (model walter/switch/pcb_push.wrl
+    (model ${P3D_WALTER}/switch/pcb_push.wrl
       (at (xyz 0 0 0))
       (scale (xyz 1 1 1))
@@
       (rotate (xyz 0 0 0))
     )
+    (model ${P3D_WALTER}/pth_circuits/dil_28-600_socket.wrl
+      (offset (xyz 7.55 -16.4 0))
+      (scale (xyz 1 1 1))
+      (rotate (xyz 0 0 -90))
+    )
   )
   (module OpenC64KernalCart:PinHeader_1x01_P2.54mm_Vertical (layer F.Cu)
@@
     (pad 1 thru_hole circle (at 0 0 270) (size 2 2) (drill 1) (layers *.Cu *.Mask)
       (net 6 VCC))
-    (pad 2 thru_hole circle (at 5 0 315) (size 2 2) (drill 1) (layers *.Cu *.Mask)
+    (pad 2 thru_hole circle (at 5 0 270) (size 2 2) (drill 1) (layers *.Cu *.Mask)
       (net 1 GND))
     (model ${KISYS3DMOD}/Capacitor_THT.3dshapes/C_Disc_D7.5mm_W2.5mm_P5.00mm.wrl
@@
     )
   )
+  (gr_arc (start 64.516 107.061) (end 64.135 107.061) (angle -90) (layer F.SilkS) (width 0.15))
+  (gr_arc (start 69.977 107.061) (end 69.977 107.442) (angle -90) (layer F.SilkS) (width 0.15))
+  (gr_arc (start 69.977 100.711) (end 70.358 100.711) (angle -90) (layer F.SilkS) (width 0.15))
+  (gr_arc (start 64.516 100.711) (end 64.516 100.33) (angle -90) (layer F.SilkS) (width 0.15))
+  (gr_line (start 64.135 107.061) (end 64.135 100.711) (layer F.SilkS) (width 0.15))
+  (gr_line (start 69.977 107.442) (end 64.516 107.442) (layer F.SilkS) (width 0.15))
+  (gr_line (start 70.358 100.711) (end 70.358 107.061) (layer F.SilkS) (width 0.15))
+  (gr_line (start 64.516 100.33) (end 69.977 100.33) (layer F.SilkS) (width 0.15))
+  (gr_text "TO CPU\nPIN 28" (at 67.31 105.537) (layer F.SilkS)
+    (effects (font (size 1 1) (thickness 0.15)))
+  )
   (gr_text A14 (at 109.22 83.439 90) (layer F.SilkS)
     (effects (font (size 1 1) (thickness 0.15)))
@@
   (via (at 62.23 96.266) (size 0.8) (drill 0.6) (layers F.Cu B.Cu) (net 1))
   (via (at 62.23 90.932) (size 0.8) (drill 0.6) (layers F.Cu B.Cu) (net 1))
-  (via (at 115.57 112.268) (size 0.8) (drill 0.6) (layers F.Cu B.Cu) (net 1))
   (via (at 115.57 96.266) (size 0.8) (drill 0.6) (layers F.Cu B.Cu) (net 1))
   (via (at 115.57 106.934) (size 0.8) (drill 0.6) (layers F.Cu B.Cu) (net 1))
   (via (at 115.57 101.6) (size 0.8) (drill 0.6) (layers F.Cu B.Cu) (net 1))
-  (via (at 115.57 117.602) (size 0.8) (drill 0.6) (layers F.Cu B.Cu) (net 1))
   (via (at 102.87 104.013) (size 0.8) (drill 0.6) (layers F.Cu B.Cu) (net 1))
   (via (at 100.33 104.013) (size 0.8) (drill 0.6) (layers F.Cu B.Cu) (net 1))
@@
   (via (at 92.71 104.8385) (size 0.8) (drill 0.6) (layers F.Cu B.Cu) (net 1))
   (via (at 80.01 107.6325) (size 0.8) (drill 0.6) (layers F.Cu B.Cu) (net 1))
-  (via (at 115.57 85.598) (size 0.8) (drill 0.6) (layers F.Cu B.Cu) (net 1))
   (via (at 115.57 90.932) (size 0.8) (drill 0.6) (layers F.Cu B.Cu) (net 1))
   (via (at 80.01 115.57) (size 0.8) (drill 0.6) (layers F.Cu B.Cu) (net 1))
@@
   (via (at 91.44 117.602) (size 0.8) (drill 0.6) (layers F.Cu B.Cu) (net 1))
   (via (at 72.39 106.076749) (size 0.8) (drill 0.6) (layers F.Cu B.Cu) (net 1))
-  (via (at 115.57 80.264) (size 0.8) (drill 0.6) (layers F.Cu B.Cu) (net 1))
-  (via (at 62.23 80.264) (size 0.8) (drill 0.6) (layers F.Cu B.Cu) (net 1))
-  (via (at 71.12 80.264) (size 0.8) (drill 0.6) (layers F.Cu B.Cu) (net 1))
   (via (at 80.01 80.264) (size 0.8) (drill 0.6) (layers F.Cu B.Cu) (net 1))
   (via (at 88.9 80.264) (size 0.8) (drill 0.6) (layers F.Cu B.Cu) (net 1))
   (via (at 97.79 80.264) (size 0.8) (drill 0.6) (layers F.Cu B.Cu) (net 1))
-  (via (at 106.68 80.264) (size 0.8) (drill 0.6) (layers F.Cu B.Cu) (net 1))
   (via (at 76.2 90.932) (size 0.8) (drill 0.6) (layers F.Cu B.Cu) (net 1))
   (via (at 81.28 90.932) (size 0.8) (drill 0.6) (layers F.Cu B.Cu) (net 1))
@@
   (via (at 95.25 98.044) (size 0.8) (drill 0.6) (layers F.Cu B.Cu) (net 1))
   (via (at 73.66 98.044) (size 0.8) (drill 0.6) (layers F.Cu B.Cu) (net 1))
-  (via (at 69.85 102.108) (size 0.8) (drill 0.6) (layers F.Cu B.Cu) (net 1))
   (via (at 107.315 104.013) (size 0.6) (drill 0.4) (layers F.Cu B.Cu) (net 1))
   (via (at 105.791 106.553) (size 0.8) (drill 0.6) (layers F.Cu B.Cu) (net 1))
@@
   (via (at 100.33 96.901) (size 0.8) (drill 0.6) (layers F.Cu B.Cu) (net 1))
   (via (at 102.87 96.901) (size 0.8) (drill 0.6) (layers F.Cu B.Cu) (net 1))
-  (segment (start 62.23 125.601726) (end 62.23 119.38) (width 0.8) (layer F.Cu) (net 1))
-  (segment (start 63.373 118.237) (end 62.23 119.38) (width 0.8) (layer F.Cu) (net 1))
-  (segment (start 63.373 116.302) (end 63.373 118.237) (width 0.8) (layer F.Cu) (net 1))
-  (segment (start 63.373 118.364) (end 62.23 119.507) (width 0.8) (layer B.Cu) (net 1))
-  (segment (start 63.373 116.302) (end 63.373 118.364) (width 0.8) (layer B.Cu) (net 1))
-  (segment (start 62.23 125.601726) (end 62.23 119.507) (width 0.8) (layer B.Cu) (net 1))
   (via (at 69.85 115.57) (size 0.8) (drill 0.6) (layers F.Cu B.Cu) (net 1))
   (via (at 69.85 112.014) (size 0.8) (drill 0.6) (layers F.Cu B.Cu) (net 1))
+  (segment (start 62.23 125.601726) (end 62.23 117.602) (width 0.8) (layer B.Cu) (net 1))
+  (segment (start 62.23 125.601726) (end 62.23 117.602) (width 0.8) (layer F.Cu) (net 1))
   (segment (start 69.85 117.602) (end 69.85 118.618) (width 0.25) (layer F.Cu) (net 2) (status 30))
   (segment (start 72.39 121.158) (end 72.39 125.601726) (width 0.25) (layer F.Cu) (net 2) (status 20))
